File: hardware/Li Ion Doctor.kicad_sch (KiCad schematic)
At the start: 37 parts, among them J1 BAT+, J2 BAT-, Q1 MMBT3906, Q2 IRFZ44N, SW1 RotaryEncoder_Switch, U1 LM358M, U2 ADS1015

Commit message: Remove some warnings
Changed lines of the file:
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@@
 (kicad_sch
-	(version 20231120)
+	(version 20250114)
 	(generator "eeschema")
-	(generator_version "8.0")
+	(generator_version "9.0")
 	(paper "A4")
 	(title_block
 		(title "Lithium battery doctor")
-		(date "2024-06-12")
+		(date "2024-10-10")
 		(rev "1")
 		(comment 1 "Modified by GMagician")
 		(comment 2 "Original project by Akos Boda")
 	)
+	(text "1W"
+		(exclude_from_sim no)
+		(at 229.362 55.372 0)
+		(effects
+			(font
+				(size 1.27 1.27)
+			)
+			(justify left bottom)
+		)
+	)
+	(text "1W"
+		(exclude_from_sim no)
+		(at 236.982 55.372 0)
+		(effects
+			(font
+				(size 1.27 1.27)
+			)
+			(justify left bottom)
+		)
+	)
+	(text "1W"
+		(exclude_from_sim no)
+		(at 244.602 55.372 0)
+		(effects
+			(font
+				(size 1.27 1.27)
+			)
+			(justify left bottom)
+		)
+	)
+	(text "1.1V"
+		(exclude_from_sim no)
+		(at 182.88 102.108 0)
+		(effects
+			(font
+				(size 1.27 1.27)
+			)
+			(justify left bottom)
+		)
+	)
+	(text_box "DISCHARGE"
+		(exclude_from_sim no)
+		(at 156.21 113.03 0)
+		(size 95.25 39.37)
+		(margins 0.9525 0.9525 0.9525 0.9525)
+		(stroke
+			(width 0)
+			(type dash)
+		)
+		(fill
+			(type none)
+		)
+		(effects
+			(font
+				(size 1.27 1.27)
+			)
+			(justify left top)
+		)
+	)
+	(text_box "RECOVERY (Optional)"
+		(exclude_from_sim no)
+		(at 102.87 33.02 0)
+		(size 34.29 33.02)
+		(margins 0.9525 0.9525 0.9525 0.9525)
+		(stroke
+			(width 0)
+			(type dash)
+		)
+		(fill
+			(type none)
+		)
+		(effects
+			(font
+				(size 1.27 1.27)
+			)
+			(justify left top)
+		)
+	)
+	(text_box "NEAR ADS POWER"
+		(exclude_from_sim no)
+		(at 146.05 48.26 0)
+		(size 24.13 17.78)
+		(margins 0.9525 0.9525 0.9525 0.9525)
+		(stroke
+			(width 0)
+			(type dash)
+		)
+		(fill
+			(type none)
+		)
+		(effects
+			(font
+				(size 1.27 1.27)
+			)
+			(justify left top)
+		)
+	)
+	(text_box "AMEASURE"
+		(exclude_from_sim no)
+		(at 180.34 68.58 0)
+		(size 46.99 40.64)
+		(margins 0.9525 0.9525 0.9525 0.9525)
+		(stroke
+			(width 0)
+			(type dash)
+		)
+		(fill
+			(type none)
+		)
+		(effects
+			(font
+				(size 1.27 1.27)
+			)
+			(justify left top)
+		)
+	)
 	(junction
 		(at 248.92 85.09)
@@
 		)
 	)
-	(text_box "DISCHARGE"
-		(exclude_from_sim no)
-		(at 156.21 113.03 0)
-		(size 95.25 39.37)
-		(stroke
-			(width 0)
-			(type dash)
-		)
-		(fill
-			(type none)
-		)
-		(effects
-			(font
-				(size 1.27 1.27)
-			)
-			(justify left top)
-		)
-	)
-	(text_box "RECOVERY (Optional)"
-		(exclude_from_sim no)
-		(at 102.87 33.02 0)
-		(size 34.29 33.02)
-		(stroke
-			(width 0)
-			(type dash)
-		)
-		(fill
-			(type none)
-		)
-		(effects
-			(font
-				(size 1.27 1.27)
-			)
-			(justify left top)
-		)
-	)
-	(text_box "NEAR ADS POWER"
-		(exclude_from_sim no)
-		(at 146.05 48.26 0)
-		(size 24.13 17.78)
-		(stroke
-			(width 0)
-			(type dash)
-		)
-		(fill
-			(type none)
-		)
-		(effects
-			(font
-				(size 1.27 1.27)
-			)
-			(justify left top)
-		)
-	)
-	(text_box "AMEASURE"
-		(exclude_from_sim no)
-		(at 180.34 68.58 0)
-		(size 46.99 40.64)
-		(stroke
-			(width 0)
-			(type dash)
-		)
-		(fill
-			(type none)
-		)
-		(effects
-			(font
-				(size 1.27 1.27)
-			)
-			(justify left top)
-		)
-	)
-	(text "1W"
-		(exclude_from_sim no)
-		(at 229.362 55.372 0)
-		(effects
-			(font
-				(size 1.27 1.27)
-			)
-			(justify left bottom)
-		)
-	)
-	(text "1W"
-		(exclude_from_sim no)
-		(at 236.982 55.372 0)
-		(effects
-			(font
-				(size 1.27 1.27)
-			)
-			(justify left bottom)
-		)
-	)
-	(text "1W"
-		(exclude_from_sim no)
-		(at 244.602 55.372 0)
-		(effects
-			(font
-				(size 1.27 1.27)
-			)
-			(justify left bottom)
-		)
-	)
-	(text "1.1V"
-		(exclude_from_sim no)
-		(at 182.88 102.108 0)
-		(effects
-			(font
-				(size 1.27 1.27)
-			)
-			(justify left bottom)
-		)
-	)
 	(label "SCL"
 		(at 49.53 175.26 0)
-		(fields_autoplaced yes)
 		(effects
 			(font
@@
 	(label "SDA"
 		(at 49.53 177.8 0)
-		(fields_autoplaced yes)
 		(effects
 			(font
@@
 	(label "~{ENCBTN}"
 		(at 96.52 170.18 0)
-		(fields_autoplaced yes)
 		(effects
 			(font
@@
 	(label "ENCA"
 		(at 73.66 170.18 180)
-		(fields_autoplaced yes)
 		(effects
 			(font
@@
 	(label "ENCB"
 		(at 96.52 105.41 180)
-		(fields_autoplaced yes)
 		(effects
 			(font
@@
 	(label "SDA"
 		(at 43.18 153.67 270)
-		(fields_autoplaced yes)
 		(effects
 			(font
@@
 	(label "ENCB"
 		(at 73.66 175.26 180)
-		(fields_autoplaced yes)
 		(effects
 			(font
@@
 	(label "~{ENCBTN}"
 		(at 96.52 102.87 180)
-		(fields_autoplaced yes)
 		(effects
 			(font
@@
 	(label "SCL"
 		(at 123.19 85.09 0)
-		(fields_autoplaced yes)
 		(effects
 			(font
@@
 	(label "SCL"
 		(at 34.29 153.67 270)
-		(fields_autoplaced yes)
 		(effects
 			(font
@@
 	(label "DISCHARGE_EN"
 		(at 233.68 130.81 0)
-		(fields_autoplaced yes)
 		(effects
 			(font
@@
 	(label "DISCHARGE_EN"
 		(at 248.92 67.31 0)
-		(fields_autoplaced yes)
 		(effects
 			(font
@@
 	(label "SDA"
 		(at 123.19 87.63 0)
-		(fields_autoplaced yes)
 		(effects
 			(font
@@
 	(label "ENCA"
 		(at 96.52 107.95 180)
-		(fields_autoplaced yes)
 		(effects
 			(font
@@
 		(at 28.575 23.495)
 		(size 13.335 13.335)
+		(exclude_from_sim no)
+		(in_bom yes)
+		(on_board yes)
+		(dnp no)
 		(stroke
 			(width 0.1524)
@@
 		)
 	)
+	(embedded_fonts no)
 )
